Commit message: Add csv file with experimental values and pose_array.py script (minichallenge 4)

File: urdf/puzzlebot_jetson_ed_urdf.urdf (robot description, URDF)
Before this commit: robot Puzzlebot Jetson-Lidar Ed., 4 links, 3 joints
Links:
- link chassis: geometry collision mesh filename=package://aranchubots_autonomousnavigation_puzzlebot/models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; visual mesh filename=package://aranchubots_autonomousnavigation_puzzlebot/models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
- link link_wl: geometry collision mesh filename=package://aranchubots_autonomousnavigation_puzzlebot/models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; visual mesh filename=package://aranchubots_autonomousnavigation_puzzlebot/models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
- link link_wr: geometry collision mesh filename=package://aranchubots_autonomousnavigation_puzzlebot/models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; visual mesh filename=package://aranchubots_autonomousnavigation_puzzlebot/models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
