Commit message: Navigation on real robot

File: urdf/puzzlebot_real.xacro (robot description, xacro)
@@ -2,7 +2,6 @@
 <!-- PuzzleBot differential drive -->
 <robot name="puzzlebot" xmlns:xacro="http://www.ros.org/wiki/xacro">
-<!-- files for gazebo costumization -->
 <xacro:include filename="$(find aranchubots_autonomousnavigation_puzzlebot)/urdf/materials.xacro" />
-<xacro:include filename="$(find aranchubots_autonomousnavigation_puzzlebot)/urdf/parameters.xacro" />
+<xacro:include filename="$(find aranchubots_autonomousnavigation_puzzlebot)/urdf/parameters_real.xacro" />
 <xacro:include filename="$(find aranchubots_autonomousnavigation_puzzlebot)/urdf/puzzlebot.gazebo" />
 <xacro:include filename="$(find aranchubots_autonomousnavigation_puzzlebot)/urdf/macros.xacro" />
@@ -193,7 +192,4 @@
     </collision>
 </link>
-<gazebo reference="base_laser_link"> <!--Color for the link -->
-    <material>Gazebo/Black</material>
-</gazebo>
 <!-- joint to attach the laser to the chassis -->
 <joint name="joint_base_laser_link" type="fixed">
@@ -202,35 +198,10 @@
 	<child link="base_laser_link"/>
 </joint>
-<!-- plugin for the laser -->
-<gazebo reference="base_laser_link">
-    <sensor type="ray" name="head_rplidar">
-        <pose>0 0 0 0 0 0</pose>
-        <visualize>false</visualize>
-        <update_rate>10</update_rate><!--10 hz as the RP lidar-->
-        <ray>
-            <scan>
-                <horizontal>
-                    <samples>1440</samples>
-                    <resolution>1</resolution>
-                    <min_angle>-3.141596</min_angle>
-                    <max_angle>3.141596</max_angle>
-                </horizontal>
-            </scan>
-            <range>
-                <min>0.15</min>
-                <max>8.0</max>
-                <resolution>0.01</resolution>
-            </range>
-            <noise>
-                <type>gaussian</type>
-                <mean>0.0</mean>
-                <stddev>0.01</stddev>
-            </noise>
-        </ray>
-        <plugin name="gazebo_ros_head_hokuyo_controller" filename="libgazebo_ros_laser.so">
-            <topicName>/scan</topicName>
-            <frameName>base_laser_link</frameName>
-        </plugin>
-    </sensor>
-</gazebo>
+<joint name="joint_laser_laser_link" type="fixed">
+	<origin xyz="0.0 0 0.0" rpy="0 0.0 3.141592"/>
+	<parent link="base_laser_link"/>
+	<child link="laser"/>
+</joint>
+<link name="laser">
+</link>
 </robot>

Commit message: Ready for real Bug2

File: urdf/puzzlebot_real.xacro (robot description, xacro)
@@ -199,5 +199,5 @@
 </joint>
 <joint name="joint_laser_laser_link" type="fixed">
-	<origin xyz="0.0 0 0.0" rpy="0 0.0 3.141592"/>
+	<origin xyz="0.0 0 0.0" rpy="0 0.0 3.14"/>
 	<parent link="base_laser_link"/>
 	<child link="laser"/>
