Commit message: Kalman Filter

File: urdf/parameters_real.xacro (robot description, xacro)
@@ -19,6 +19,6 @@
 <xacro:property name="cameraY" value="0.04"/>
 <xacro:property name="cameraZ" value="0.06"/>
-<xacro:property name="mesh_chassis"  value="/home/estebanpadilla/catkin_ws/src/aranchubots_autonomousnavigation_puzzlebot/meshes/chassis.stl" />
-<xacro:property name="mesh_wheel"  value="/home/estebanpadilla/catkin_ws/src/aranchubots_autonomousnavigation_puzzlebot/meshes/wheel.stl" />
-<xacro:property name="mesh_camera"  value="/home/estebanpadilla/catkin_ws/src/aranchubots_autonomousnavigation_puzzlebot/meshes/camera.stl" />
+<xacro:property name="mesh_chassis"  value="/home/esteb37/catkin_ws/src/aranchubots_autonomousnavigation_puzzlebot/meshes/chassis.stl" />
+<xacro:property name="mesh_wheel"  value="/home/esteb37/catkin_ws/src/aranchubots_autonomousnavigation_puzzlebot/meshes/wheel.stl" />
+<xacro:property name="mesh_camera"  value="/home/esteb37/catkin_ws/src/aranchubots_autonomousnavigation_puzzlebot/meshes/camera.stl" />
 </robot>

Commit message: Sim map with markers and real ready

File: urdf/parameters_real.xacro (robot description, xacro)
@@ -19,6 +19,6 @@
 <xacro:property name="cameraY" value="0.04"/>
 <xacro:property name="cameraZ" value="0.06"/>
-<xacro:property name="mesh_chassis"  value="/home/esteb37/catkin_ws/src/aranchubots_autonomousnavigation_puzzlebot/meshes/chassis.stl" />
-<xacro:property name="mesh_wheel"  value="/home/esteb37/catkin_ws/src/aranchubots_autonomousnavigation_puzzlebot/meshes/wheel.stl" />
-<xacro:property name="mesh_camera"  value="/home/esteb37/catkin_ws/src/aranchubots_autonomousnavigation_puzzlebot/meshes/camera.stl" />
+<xacro:property name="mesh_chassis"  value="/home/estebanpadilla/catkin_ws/src/aranchubots_autonomousnavigation_puzzlebot/meshes/chassis.stl" />
+<xacro:property name="mesh_wheel"  value="/home/estebanpadilla/catkin_ws/src/aranchubots_autonomousnavigation_puzzlebot/meshes/wheel.stl" />
+<xacro:property name="mesh_camera"  value="/home/estebanpadilla/catkin_ws/src/aranchubots_autonomousnavigation_puzzlebot/meshes/camera.stl" />
 </robot>
